Commit message: add urdf for lb

File: urdf/materials.urdf.xacro (robot description, xacro)
@@ -16,4 +16,7 @@
     <color rgba="0.0 0.0 0.0 1.0"/>
   </material>
+  <material name="Black">
+    <color rgba="0.0 0.0 0.0 1.0"/>
+  </material>
   <material name="youBot/Red">
     <color rgba="1.0 0.0 0.0 1.0"/>

File: urdf/youbot_arm/arm.urdf.xacro (robot description, xacro)
@@ -39,5 +39,5 @@
 		<!-- joint between arm_0_link and arm_1_link -->
 		<joint name="${name}_joint_1" type="revolute">
-			<origin xyz="0.024 0 0.096" rpy="0 0 ${170 * M_PI / 180}"/>
+			<origin xyz="0.024 0 0.096" rpy="0 0 ${170 * M_PI / 180 - 0.04}"/>
 			<parent link="${name}_link_0"/>
 			<child link="${name}_link_1"/>
@@ -47,5 +47,5 @@
 			<!-- damping - N*s/m, N*s*m/rad -->
 			<!-- friction - N, N*m -->
-			<limit effort="${9.5}" velocity="${M_PI / 2.0}" lower="0" upper="${joint_1_limit}"/>
+			<limit effort="${9.5}" velocity="${M_PI / 2.0}" lower="${joint_1_limit_lower}" upper="${joint_1_limit_upper}"/>
 			<!--effort - N, N*m-->
 			<!--velocity - m/s, rad/s-->
@@ -78,5 +78,5 @@
 		<!-- joint between arm_1_link and arm_2_link -->
 		<joint name="${name}_joint_2" type="revolute">
-			<origin xyz="0.033 0 0.019" rpy="0 ${-65 * M_PI / 180} 0"/>
+			<origin xyz="0.033 0 0.019" rpy="0 ${-65 * M_PI / 180 + 0.04} 0"/>
 			<parent link="${name}_link_1"/>
 			<child link="${name}_link_2"/>
@@ -84,5 +84,5 @@
 			<!--<calibration rising="${arm_2_ref}" falling="${arm_2_ref}"/>-->
 			<dynamics damping="1" friction="0.5" />
-			<limit effort="${9.5}" velocity="${M_PI / 2.0}" lower="0" upper="${joint_2_limit}"/>
+			<limit effort="${9.5}" velocity="${M_PI / 2.0}" lower="${joint_2_limit_lower}" upper="${joint_2_limit_upper}"/>
       <!--safety_controller k_position="20" k_velocity="${2*9.5/M_PI}" soft_lower_limit="${threshold}" soft_upper_limit="${joint_2_limit_soft}" /-->
 		</joint>
@@ -118,10 +118,10 @@
 		</joint>-->
 		<joint name="${name}_joint_3" type="revolute">
-			<origin xyz="0.000 0.000 0.155" rpy="0 ${146 * M_PI / 180} 0"/>
+			<origin xyz="0.000 0.000 0.155" rpy="0 ${146 * M_PI / 180 - 0.04} 0"/>
 			<parent link="${name}_link_2"/>
 			<child link="${name}_link_3"/>
 			<axis xyz="0 1 0"/>
 			<dynamics damping="1" friction="0.5" />
-			<limit effort="${6.0}" velocity="${M_PI / 2.0}" lower="-${joint_3_limit}" upper="0"/>
+			<limit effort="${6.0}" velocity="${M_PI / 2.0}" lower="${joint_3_limit_lower}" upper="${joint_3_limit_upper}"/>
       <!--safety_controller k_position="20" k_velocity="50" soft_lower_limit="-${joint_3_limit_soft}" soft_upper_limit="-${threshold}" /-->
 		</joint>
@@ -149,5 +149,5 @@
 		<!-- joint between arm_3_link and arm_4_link -->
 		<joint name="${name}_joint_4" type="revolute">
-			<origin xyz="0.000 0.000 0.135" rpy="0 ${-102.5 * M_PI / 180} 0" />
+			<origin xyz="0.000 0.000 0.135" rpy="0 ${-102.5 * M_PI / 180 + 0.04} 0" />
 			<parent link="${name}_link_3"/>
 			<child link="${name}_link_4"/>
@@ -155,5 +155,5 @@
 			<!--<calibration rising="${arm_4_ref}" falling="${arm_4_ref}"/>-->
 			<dynamics damping="1" friction="0.5" />
-			<limit effort="${2.0}" velocity="${M_PI / 2.0}" lower="0" upper="${joint_4_limit}"/>
+			<limit effort="${2.0}" velocity="${M_PI / 2.0}" lower="${joint_4_limit_lower}" upper="${joint_4_limit_upper}"/>
 			<!--safety_controller k_position="20" k_velocity="100" soft_lower_limit="0" soft_upper_limit="${joint_4_limit_soft}" /-->
 		</joint>
@@ -181,5 +181,5 @@
 		<!-- joint between arm_4_link and arm_5_link -->
 		<joint name="${name}_joint_5" type="revolute">
-			<origin xyz="-0.002 0 0.130" rpy="0 0 ${167.5 * M_PI / 180}" />
+			<origin xyz="-0.002 0 0.130" rpy="0 0 ${167.5 * M_PI / 180 + 0.04}" />
 			<parent link="${name}_link_4"/>
 			<child link="${name}_link_5"/>
@@ -187,5 +187,5 @@
 			<!--<calibration rising="${arm_5_ref}" falling="${arm_5_ref}"/>-->
 			<dynamics damping="0.5" friction="0.5" />
-			<limit effort="${1.0}" velocity="${M_PI / 2.0}" lower="0" upper="${joint_5_limit}" />
+			<limit effort="${1.0}" velocity="${M_PI / 2.0}" lower="${joint_5_limit_lower}" upper="${joint_5_limit_upper}" />
       <!--safety_controller k_position="20" k_velocity="100" soft_lower_limit="0" soft_upper_limit="${joint_5_limit_soft}" /-->
 		</joint>

File: urdf/youbot_arm/limits.urdf.xacro (robot description, xacro)
@@ -3,5 +3,5 @@
 	<!-- common properties -->
 	<xacro:property name="M_PI" value="3.1415926535897931" />
-	<xacro:property name="threshold" value="0.01" />
+	<xacro:property name="threshold" value="1" />
 	<!-- arm limits positions (deg) -->
 	<xacro:property name="joint_1_limit" value="${M_PI * (169 + 169) / 180}" />
@@ -15,4 +15,14 @@
 	<xacro:property name="joint_4_limit_soft" value="${joint_4_limit - threshold}" />
 	<xacro:property name="joint_5_limit_soft" value="${joint_5_limit - threshold}" />
+	<xacro:property name="joint_1_limit_upper" value="${5.84014 - 0.03}" />
+	<xacro:property name="joint_2_limit_upper" value="${2.61799 - 0.03}" />
+	<xacro:property name="joint_3_limit_upper" value="${-0.0157 - 0.03}" />
+	<xacro:property name="joint_4_limit_upper" value="${3.4292  - 0.03}" />
+	<xacro:property name="joint_5_limit_upper" value="${5.64159 - 0.03}" />
+	<xacro:property name="joint_1_limit_lower" value="${0.0100692 + 0.03}" />
+	<xacro:property name="joint_2_limit_lower" value="${0.0100692 + 0.03}" />
+	<xacro:property name="joint_3_limit_lower" value="${-5.02655  + 0.03}" />
+	<xacro:property name="joint_4_limit_lower" value="${0.0221239 + 0.03}" />
+	<xacro:property name="joint_5_limit_lower" value="${0.110619  + 0.03}" />
 	<!-- dynamic properties : mass (kg) Alu data sheet -->
 	<xacro:property name="link_0_mass" value="0.961" />
